File: hardware/kicad/KOGUMA-Mk4/power.kicad_sch (KiCad schematic)
At the start: 21 parts, among them J1 BATT (BT2.0), Q1 AO4407A, SW1 SSSS810701, U1 LXDC55FAAA-203

Commit message: SW1・SW2・BZ1 のフットプリントを作り、NJU6080 を SOT-23-6 に。全部の部品にフットプリントが付いた
寸法はメーカーの推奨ランド: SSSS810701(Alps の Land Dimensions)、TVAF06-A020B-R(仕様書の
P.C.B LAND DIMENSION)、SMT-0540-S-R(Suggested Land Pattern)。gen_footprints.py で作る。ERC エラー 0

Co-Authored-By: Claude Opus 5.5 <noreply@anthropic.com>
Claude-Session: https://claude.ai/code/session_01H2Zvpqxqu2v63zaiCMmfT3
Parts:
- SW1: footprint (none) -> KOGUMA-Mk4:SW_Slide_SPDT_Alps_SSSS8
Changed lines of the file:
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@@
 			)
 		)
-		(property "Footprint" ""
+		(property "Footprint" "KOGUMA-Mk4:SW_Slide_SPDT_Alps_SSSS8"
 			(at 96.52 54.61 0)
 			(effects
